Commit message: urdf changes

File: urdf/relife_model.urdf.xacro (robot description, xacro)
@@ -44,4 +44,11 @@
       <origin xyz="0 0 0" rpy="0 0 0"/>
     </xacro:inertial_box>
+    <xacro:inertial_box
+      mass="85.0"
+      x="0.45"
+      y="0.28"
+      z="0.18">
+      <origin xyz="0 0 0.09" rpy="0 0 0"/>
+    </xacro:inertial_box>
   </link>
   <!-- Odom Frame -->
@@ -53,5 +60,4 @@
     <origin xyz="0 0 0" rpy="0 0 0"/>
   </joint>
-  <!-- Body link - increased mass from 1.0 to 20.0 kg -->
   <link name="Body_link">
     <collision>
@@ -61,7 +67,11 @@
         </geometry>
     </collision>
-    <xacro:inertial_box mass="20.0" x="0.45" y="0.28" z="0.18">
-      <origin xyz="0.17 0.0 0.15" rpy="0.0 0.0 0.0"/>
-    </xacro:inertial_box>
+    <xacro:inertial_box
+      mass="85.0"
+      x="0.45"
+      y="0.28"
+      z="0.18">
+      <origin xyz="0 0 0.09" rpy="0 0 0" />
+  </xacro:inertial_box>
     <visual>
         <origin rpy="0.0 1.42294 0.0" xyz="0.17482 -0.00088 0.15732"/>
@@ -77,24 +87,23 @@
       <origin xyz="0 0 0" rpy="0 0 0"/>
   </joint>
-  <!-- Wheel joints - keep orientation but adjust dynamics -->
-  <joint name="BackWheel_link_joint" type="fixed">
-    <limit lower="0" upper="1" effort="100" velocity="0.50"/>
-    <origin rpy="${pi/2} 0 0" xyz="-0.45842 0.00285 0.05"/>
+  <joint name="BackWheel_link_joint" type="revolute">
     <parent link="Body_link"/>
     <child link="BackWheel_link"/>
+    <origin xyz="-0.45842 0.00285 0.05" rpy="${pi/2} 0 0"/>
     <axis xyz="0 0 1"/>
-    <dynamics damping="0.5" friction="0.1"/>  <!-- Increased damping and friction -->
-  </joint>
-  <joint name="FrontWheel_link_joint" type="fixed">
-    <limit lower="0" upper="1" effort="100" velocity="0.50"/>
-    <origin rpy="${pi/2} 0 0" xyz="0.17030 0.00221 0.05"/>
+    <limit lower="-1e16" upper="1e16" effort="1.0" velocity="10.0"/>
+    <dynamics damping="0.0" friction="0.0"/>
+  </joint>
+  <joint name="FrontWheel_link_joint" type="revolute">
     <parent link="Body_link"/>
     <child link="FrontWheel_link"/>
+    <origin xyz="0.17030 0.00221 0.05" rpy="${pi/2} 0 0"/>
     <axis xyz="0 0 1"/>
-    <dynamics damping="0.5" friction="0.1"/>  <!-- Increased damping and friction -->
+    <limit lower="-1e16" upper="1e16" effort="1.0" velocity="10.0"/>
+    <dynamics damping="0.0" friction="0.0"/>
   </joint>
   <!-- Driving wheels - increased effort and adjusted dynamics -->
   <joint name="LeftWheel_link_joint" type="continuous">
-    <limit effort="50" velocity="0.5"/>  <!-- Increased effort from 10 to 50 -->
+    <limit effort="250" velocity="0.5"/>  <!-- Increased effort from 10 to 50 -->
     <dynamics damping="0.1" friction="0.1"/>  <!-- Increased damping and friction -->
     <origin rpy="${-pi/2} 0 0" xyz="-0.24508 0.28586 0.05"/>
@@ -102,7 +111,8 @@
     <child link="LeftWheel_link"/>
     <axis xyz="0 0 1"/>
+    <dynamics damping="5.0" friction="0.1"/>
   </joint>
   <joint name="RightWheel_link_joint" type="continuous">
-    <limit effort="50" velocity="0.5"/>  <!-- Increased effort from 10 to 50 -->
+    <limit effort="250" velocity="0.5"/>  <!-- Increased effort from 10 to 50 -->
     <dynamics damping="0.1" friction="0.1"/>  <!-- Increased damping and friction -->
     <origin rpy="${pi/2} 0 0" xyz="-0.24508 -0.28586 0.05"/>
@@ -110,4 +120,5 @@
     <child link="RightWheel_link"/>
     <axis xyz="0 0 -1"/>
+    <dynamics damping="5.0" friction="0.1"/>
   </joint>
   <!-- Wheels - increased mass from 0.5 to 3.75 kg each -->
@@ -120,7 +131,10 @@
       </geometry>
     </collision>
-    <xacro:inertial_cylinder mass="3.75" length="0.02" radius="0.05">
-      <origin xyz="0 0 0" rpy="0 0 0"/>
-    </xacro:inertial_cylinder>
+    <xacro:inertial_cylinder
+    mass="3.75"
+    length="0.02"
+    radius="0.05">
+    <origin xyz="-0.45842 0.00285 0.05" rpy="${pi/2} 0 0"/>
+  </xacro:inertial_cylinder>
     <visual name="BackWheel">
       <origin xyz="0 0 0" rpy="${pi/2} 0 ${pi/2}"/>
@@ -139,7 +153,10 @@
       </geometry>
     </collision>
-    <xacro:inertial_cylinder mass="3.75" length="0.02" radius="0.05">
-      <origin xyz="0 0 0" rpy="0 0 0"/>
-    </xacro:inertial_cylinder>
+    <xacro:inertial_cylinder
+    mass="3.75"
+    length="0.02"
+    radius="0.05">
+    <origin xyz="-0.45842 0.00285 0.05" rpy="${pi/2} 0 0"/>
+  </xacro:inertial_cylinder>
     <visual name="FrontWheel">
       <origin xyz="0 0 0" rpy="${pi/2} 0 ${pi/2}"/>
@@ -158,7 +175,4 @@
       </geometry>
     </collision>
-    <xacro:inertial_cylinder mass="3.75" length="0.02" radius="0.05">
-      <origin xyz="0 0 0" rpy="0 0 0"/>
-    </xacro:inertial_cylinder>
     <visual name="LeftWheel">
       <origin xyz="0 0 0" rpy="${-pi/2} 0 ${pi/2}"/>
@@ -168,4 +182,24 @@
       </geometry>
     </visual>
+    <xacro:inertial_cylinder
+    mass="3.75"
+    length="0.02"
+    radius="0.05">
+    <origin xyz="-0.45842 0.00285 0.05" rpy="${pi/2} 0 0"/>
+  </xacro:inertial_cylinder>
+    <collision>
+      <geometry>
+        <cylinder radius="0.05" length="0.02"/>
+      </geometry>
+      <surface>
+        <friction>
+          <ode>
+            <mu>0.8</mu>    <!-- sliding friction -->
+            <mu2>0.4</mu2>  <!-- rolling friction -->
+          </ode>
+        </friction>
+        <!-- optional bounce, contact parameters, etc. -->
+      </surface>
+    </collision>
   </link>
   <!-- Right Wheel -->
@@ -177,7 +211,4 @@
       </geometry>
     </collision>
-    <xacro:inertial_cylinder mass="3.75" length="0.02" radius="0.05">
-      <origin xyz="0 0 0" rpy="0 0 0"/>
-    </xacro:inertial_cylinder>
     <visual name="RightWheel">
       <origin xyz="0 0 0" rpy="${pi/2} 0 ${pi/2}"/>
@@ -187,4 +218,24 @@
       </geometry>
     </visual>
+    <xacro:inertial_cylinder
+    mass="3.75"
+    length="0.02"
+    radius="0.05">
+    <origin xyz="-0.45842 0.00285 0.05" rpy="${pi/2} 0 0"/>
+  </xacro:inertial_cylinder>
+    <collision>
+      <geometry>
+        <cylinder radius="0.05" length="0.02"/>
+      </geometry>
+      <surface>
+        <friction>
+          <ode>
+            <mu>0.8</mu>    <!-- sliding friction -->
+            <mu2>0.4</mu2>  <!-- rolling friction -->
+          </ode>
+        </friction>
+        <!-- optional bounce, contact parameters, etc. -->
+      </surface>
+    </collision>
   </link>
   <!-- Ultrasonic sensor - unchanged -->
@@ -273,25 +324,24 @@
     <color rgba="0.10588 0.10588 0.10588 1.0"/>
   </material>
-  <!-- Gazebo specific properties - adjusted for 50kg robot -->
   <gazebo reference="LeftWheel_link">
-    <mu1>1.5</mu1>  <!-- Increased from 1.0 for better traction -->
-    <mu2>1.5</mu2>  <!-- Increased from 1.0 for better traction -->
-    <kp>1000000.0</kp>
-    <kd>100.0</kd>
-    <max_vel>1.0</max_vel>  <!-- Increased from 0.2 -->
-    <max_force>250.0</max_force>  <!-- Increased from 10.0 -->
+    <mu1>2.0</mu1>  <!-- Slightly reduced from 2.5 -->
+    <mu2>2.0</mu2>  <!-- Slightly reduced from 2.5 -->
+    <kp>250.0</kp>  <!-- Reduced from 500.0 -->
+    <kd>5.0</kd>    <!-- Reduced from 10.0 -->
+    <max_vel>0.5</max_vel>  <!-- Reduced from 1.0 -->
+    <max_force>100.0</max_force>  <!-- Reduced from 250.0 -->
   </gazebo>
   <gazebo reference="RightWheel_link">
-    <mu1>1.5</mu1>  <!-- Increased from 1.0 for better traction -->
-    <mu2>1.5</mu2>  <!-- Increased from 1.0 for better traction -->
-    <kp>1000000.0</kp>
-    <kd>100.0</kd>
-    <max_vel>1.0</max_vel>  <!-- Increased from 0.2 -->
-    <max_force>250.0</max_force>  <!-- Increased from 10.0 -->
+    <mu1>2.0</mu1>  <!-- Slightly reduced from 2.5 -->
+    <mu2>2.0</mu2>  <!-- Slightly reduced from 2.5 -->
+    <kp>250.0</kp>  <!-- Reduced from 500.0 -->
+    <kd>5.0</kd>    <!-- Reduced from 10.0 -->
+    <max_vel>0.5</max_vel>  <!-- Reduced from 1.0 -->
+    <max_force>100.0</max_force>  <!-- Reduced from 250.0 -->
   </gazebo>
   <gazebo reference="FrontWheel_link">
     <mu1>0.1</mu1>  <!-- Lowered from 0.2 for better sliding -->
     <mu2>0.1</mu2>  <!-- Lowered from 0.2 for better sliding -->
-    <kp>100000.0</kp>  <!-- Increased for better stability -->
+    <kp>10.0</kp>  <!-- Increased for better stability -->
     <kd>10.0</kd>  <!-- Increased for better stability -->
   </gazebo>
@@ -299,5 +349,5 @@
     <mu1>0.1</mu1>  <!-- Lowered from 0.2 for better sliding -->
     <mu2>0.1</mu2>  <!-- Lowered from 0.2 for better sliding -->
-    <kp>100000.0</kp>  <!-- Increased for better stability -->
+    <kp>10.0</kp>  <!-- Increased for better stability -->
     <kd>10.0</kd>  <!-- Increased for better stability -->
   </gazebo>
@@ -340,6 +390,7 @@
       <wheel_separation>0.57</wheel_separation>
       <wheel_diameter>0.1</wheel_diameter>
-      <max_wheel_torque>100</max_wheel_torque>  <!-- Increased from 20 -->
-      <max_wheel_acceleration>0.3</max_wheel_acceleration>  <!-- Reduced from 0.5 for smoother movement -->
+      <max_wheel_torque>75</max_wheel_torque>  <!-- Reduced from 150 to prevent tipping -->
+      <max_wheel_acceleration>0.05</max_wheel_acceleration>  <!-- Significantly reduced to prevent tipping -->
+      <max_velocity>0.3</max_velocity>  <!-- Moderate top speed -->
       <publish_odom>true</publish_odom>
       <publish_odom_tf>true</publish_odom_tf>

File: urdf/relife_ros2_control.xacro (robot description, xacro)
@@ -12,4 +12,11 @@
             <state_interface name="position" />
             <state_interface name="velocity" />
+            <parameters>
+                <pid>
+                  <p>5.0</p>    <!-- proportional gain -->
+                  <i>0.1</i>    <!-- integral gain, often zero for velocity -->
+                  <d>0.01</d>   <!-- derivative gain -->
+                </pid>
+              </parameters>
         </joint>
         <joint name="LeftWheel_link_joint">
@@ -20,4 +27,11 @@
             <state_interface name="position" />
             <state_interface name="velocity" />
+            <parameters>
+                <pid>
+                  <p>5.0</p>    <!-- proportional gain -->
+                  <i>0.1</i>    <!-- integral gain, often zero for velocity -->
+                  <d>0.01</d>   <!-- derivative gain -->
+                </pid>
+              </parameters>
         </joint>
     </ros2_control>
@@ -29,5 +43,5 @@
         <joint name="RightWheel_link_joint">
             <hardwareInterface>hardware_interface/velocity</hardwareInterface>
-            <mechanical_reduction>10.0</mechanical_reduction>  <!-- Increased from 1.0 for better torque -->
+            <mechanical_reduction>3.0</mechanical_reduction>  <!-- Further reduced from 5.0 -->
         </joint>
     </transmission>
@@ -39,5 +53,5 @@
         <joint name="LeftWheel_link_joint">
             <hardwareInterface>hardware_interface/velocity</hardwareInterface>
-            <mechanical_reduction>10.0</mechanical_reduction>  <!-- Increased from 1.0 for better torque -->
+            <mechanical_reduction>3.0</mechanical_reduction>  <!-- Further reduced from 5.0 -->
         </joint>
     </transmission>

Commit message: updated urdf

File: urdf/relife_model.urdf.xacro (robot description, xacro)
@@ -87,5 +87,5 @@
       <origin xyz="0 0 0" rpy="0 0 0"/>
   </joint>
-  <joint name="BackWheel_link_joint" type="revolute">
+  <joint name="BackWheel_link_joint" type="fixed">
     <parent link="Body_link"/>
     <child link="BackWheel_link"/>
@@ -95,5 +95,5 @@
     <dynamics damping="0.0" friction="0.0"/>
   </joint>
-  <joint name="FrontWheel_link_joint" type="revolute">
+  <joint name="FrontWheel_link_joint" type="fixed">
     <parent link="Body_link"/>
     <child link="FrontWheel_link"/>
@@ -390,7 +390,7 @@
       <wheel_separation>0.57</wheel_separation>
       <wheel_diameter>0.1</wheel_diameter>
-      <max_wheel_torque>75</max_wheel_torque>  <!-- Reduced from 150 to prevent tipping -->
-      <max_wheel_acceleration>0.05</max_wheel_acceleration>  <!-- Significantly reduced to prevent tipping -->
-      <max_velocity>0.3</max_velocity>  <!-- Moderate top speed -->
+      <max_wheel_torque>90</max_wheel_torque>  <!-- Reduced from 150 to prevent tipping -->
+      <max_wheel_acceleration>0.1</max_wheel_acceleration>  <!-- Significantly reduced to prevent tipping -->
+      <max_velocity>1.0</max_velocity>  <!-- Moderate top speed -->
       <publish_odom>true</publish_odom>
       <publish_odom_tf>true</publish_odom_tf>

Commit message: slowly moving - needs to be faster

File: urdf/relife_model.urdf.xacro (robot description, xacro)
@@ -41,7 +41,7 @@
       </geometry>
     </collision>
-    <xacro:inertial_box mass="15.0" x="0.3" y="0.3" z="0.1">
+    <!-- <xacro:inertial_box mass="15.0" x="0.3" y="0.3" z="0.1">
       <origin xyz="0 0 0" rpy="0 0 0"/>
-    </xacro:inertial_box>
+    </xacro:inertial_box> -->
     <xacro:inertial_box
       mass="85.0"
@@ -87,24 +87,23 @@
       <origin xyz="0 0 0" rpy="0 0 0"/>
   </joint>
-  <joint name="BackWheel_link_joint" type="fixed">
+  <joint name="BackWheel_link_joint" type="revolute">
     <parent link="Body_link"/>
     <child link="BackWheel_link"/>
     <origin xyz="-0.45842 0.00285 0.05" rpy="${pi/2} 0 0"/>
     <axis xyz="0 0 1"/>
-    <limit lower="-1e16" upper="1e16" effort="1.0" velocity="10.0"/>
+    <limit effort="5" velocity="5"/>
     <dynamics damping="0.0" friction="0.0"/>
   </joint>
-  <joint name="FrontWheel_link_joint" type="fixed">
+  <joint name="FrontWheel_link_joint" type="revolute">
     <parent link="Body_link"/>
     <child link="FrontWheel_link"/>
     <origin xyz="0.17030 0.00221 0.05" rpy="${pi/2} 0 0"/>
     <axis xyz="0 0 1"/>
-    <limit lower="-1e16" upper="1e16" effort="1.0" velocity="10.0"/>
+    <limit effort="5" velocity="5"/>
     <dynamics damping="0.0" friction="0.0"/>
   </joint>
   <!-- Driving wheels - increased effort and adjusted dynamics -->
   <joint name="LeftWheel_link_joint" type="continuous">
-    <limit effort="250" velocity="0.5"/>  <!-- Increased effort from 10 to 50 -->
-    <dynamics damping="0.1" friction="0.1"/>  <!-- Increased damping and friction -->
+    <limit effort="250" velocity="50"/>  <!-- Increased effort from 10 to 50 -->
     <origin rpy="${-pi/2} 0 0" xyz="-0.24508 0.28586 0.05"/>
     <parent link="Body_link"/>
@@ -114,6 +113,5 @@
   </joint>
   <joint name="RightWheel_link_joint" type="continuous">
-    <limit effort="250" velocity="0.5"/>  <!-- Increased effort from 10 to 50 -->
-    <dynamics damping="0.1" friction="0.1"/>  <!-- Increased damping and friction -->
+    <limit effort="250" velocity="50"/>  <!-- Increased effort from 10 to 50 -->
     <origin rpy="${pi/2} 0 0" xyz="-0.24508 -0.28586 0.05"/>
     <parent link="Body_link"/>
@@ -325,18 +323,24 @@
   </material>
   <gazebo reference="LeftWheel_link">
-    <mu1>2.0</mu1>  <!-- Slightly reduced from 2.5 -->
-    <mu2>2.0</mu2>  <!-- Slightly reduced from 2.5 -->
-    <kp>250.0</kp>  <!-- Reduced from 500.0 -->
-    <kd>5.0</kd>    <!-- Reduced from 10.0 -->
-    <max_vel>0.5</max_vel>  <!-- Reduced from 1.0 -->
-    <max_force>100.0</max_force>  <!-- Reduced from 250.0 -->
+    <!-- Slightly increase friction to improve traction -->
+    <mu1>2.2</mu1>  <!-- Increased from 2.0 -->
+    <mu2>2.2</mu2>  <!-- Increased from 2.0 -->
+    <!-- Keep stiffness moderate -->
+    <kp>250.0</kp>  <!-- Keep same as original -->
+    <kd>5.0</kd>    <!-- Keep same as original -->
+    <!-- Moderate increase in velocity and force limits -->
+    <max_vel>0.9</max_vel>  <!-- Increased from 0.5 -->
+    <max_force>120.0</max_force>  <!-- Increased from 100.0 -->
   </gazebo>
   <gazebo reference="RightWheel_link">
-    <mu1>2.0</mu1>  <!-- Slightly reduced from 2.5 -->
-    <mu2>2.0</mu2>  <!-- Slightly reduced from 2.5 -->
-    <kp>250.0</kp>  <!-- Reduced from 500.0 -->
-    <kd>5.0</kd>    <!-- Reduced from 10.0 -->
-    <max_vel>0.5</max_vel>  <!-- Reduced from 1.0 -->
-    <max_force>100.0</max_force>  <!-- Reduced from 250.0 -->
+    <!-- Slightly increase friction to improve traction -->
+    <mu1>2.2</mu1>  <!-- Increased from 2.0 -->
+    <mu2>2.2</mu2>  <!-- Increased from 2.0 -->
+    <!-- Keep stiffness moderate -->
+    <kp>250.0</kp>  <!-- Keep same as original -->
+    <kd>5.0</kd>    <!-- Keep same as original -->
+    <!-- Moderate increase in velocity and force limits -->
+    <max_vel>0.9</max_vel>  <!-- Increased from 0.5 -->
+    <max_force>120.0</max_force>  <!-- Increased from 100.0 -->
   </gazebo>
   <gazebo reference="FrontWheel_link">
@@ -390,7 +394,10 @@
       <wheel_separation>0.57</wheel_separation>
       <wheel_diameter>0.1</wheel_diameter>
-      <max_wheel_torque>90</max_wheel_torque>  <!-- Reduced from 150 to prevent tipping -->
-      <max_wheel_acceleration>0.1</max_wheel_acceleration>  <!-- Significantly reduced to prevent tipping -->
-      <max_velocity>1.0</max_velocity>  <!-- Moderate top speed -->
+      <!-- Moderate increase of torque from 110 to 130 -->
+      <max_wheel_torque>130</max_wheel_torque>
+      <!-- Moderate increase from 1.0 to 1.5 -->
+      <max_wheel_acceleration>1.5</max_wheel_acceleration>
+      <!-- Moderate increase from 50.0 to 65.0 -->
+      <max_velocity>65.0</max_velocity>
       <publish_odom>true</publish_odom>
       <publish_odom_tf>true</publish_odom_tf>

File: urdf/relife_ros2_control.xacro (robot description, xacro)
@@ -7,6 +7,6 @@
         <joint name="RightWheel_link_joint">
             <command_interface name="velocity">
-                <param name="min">-2.0</param>  <!-- Increased range from -1 to -2 -->
-                <param name="max">2.0</param>   <!-- Increased range from 1 to 2 -->
+                <param name="min">-150.0</param>  <!-- Increased range from -1 to -2 -->
+                <param name="max">150.0</param>   <!-- Increased range from 1 to 2 -->
             </command_interface>
             <state_interface name="position" />
@@ -14,14 +14,14 @@
             <parameters>
                 <pid>
-                  <p>5.0</p>    <!-- proportional gain -->
-                  <i>0.1</i>    <!-- integral gain, often zero for velocity -->
-                  <d>0.01</d>   <!-- derivative gain -->
-                </pid>
+                    <p>15.0</p>    <!-- Moderately increased from 10.0 -->
+                    <i>0.2</i>     <!-- Moderately increased from 0.1 -->
+                    <d>0.02</d>    <!-- Moderately increased from 0.01 -->
+                  </pid>
               </parameters>
         </joint>
         <joint name="LeftWheel_link_joint">
             <command_interface name="velocity">
-                <param name="min">-2.0</param>  <!-- Increased range from -1 to -2 -->
-                <param name="max">2.0</param>   <!-- Increased range from 1 to 2 -->
+                <param name="min">-150.0</param>
+                <param name="max">150.0</param>
             </command_interface>
             <state_interface name="position" />
@@ -29,8 +29,8 @@
             <parameters>
                 <pid>
-                  <p>5.0</p>    <!-- proportional gain -->
-                  <i>0.1</i>    <!-- integral gain, often zero for velocity -->
-                  <d>0.01</d>   <!-- derivative gain -->
-                </pid>
+                    <p>15.0</p>    <!-- Moderately increased from 10.0 -->
+                    <i>0.2</i>     <!-- Moderately increased from 0.1 -->
+                    <d>0.02</d>    <!-- Moderately increased from 0.01 -->
+                  </pid>
               </parameters>
         </joint>
@@ -43,5 +43,5 @@
         <joint name="RightWheel_link_joint">
             <hardwareInterface>hardware_interface/velocity</hardwareInterface>
-            <mechanical_reduction>3.0</mechanical_reduction>  <!-- Further reduced from 5.0 -->
+            <mechanical_reduction>2.5</mechanical_reduction>  <!-- Further reduced from 5.0 -->
         </joint>
     </transmission>
@@ -53,5 +53,5 @@
         <joint name="LeftWheel_link_joint">
             <hardwareInterface>hardware_interface/velocity</hardwareInterface>
-            <mechanical_reduction>3.0</mechanical_reduction>  <!-- Further reduced from 5.0 -->
+            <mechanical_reduction>2.5</mechanical_reduction>  <!-- Further reduced from 5.0 -->
         </joint>
     </transmission>
