Commit message: changes and issues introduced - robot doesn't move in gazebo, but moves in rviz

File: urdf/relife_model.urdf.xacro (robot description, xacro)
@@ -2,26 +2,26 @@
 <robot xmlns:xacro="http://ros.org/wiki/xacro" name="relife">
   <!-- Include the ROS2 control configuration -->
-  <xacro:include filename="$(find re4life_robot_description)/urdf/relife_ros2_control.xacro"/>
+  <xacro:include filename="$(find re4life_robot_description)/urdf/relife_ros2_control.xacro" />
   <!-- Inertial macros - unchanged -->
   <xacro:macro name="inertial_box" params="mass x y z *origin">
     <inertial>
-      <xacro:insert_block name="origin"/>
+      <xacro:insert_block name="origin" />
       <mass value="${mass}" />
       <inertia ixx="${(1/12.0) * mass * (y*y+z*z)}"
-              ixy="0.0" ixz="0.0"
-              iyy="${(1/12.0) * mass * (x*x+z*z)}"
-              iyz="0.0"
-              izz="${(1/12.0) * mass * (x*x+y*y)}" />
+        ixy="0.0" ixz="0.0"
+        iyy="${(1/12.0) * mass * (x*x+z*z)}"
+        iyz="0.0"
+        izz="${(1/12.0) * mass * (x*x+y*y)}" />
     </inertial>
   </xacro:macro>
   <xacro:macro name="inertial_cylinder" params="mass length radius *origin">
     <inertial>
-      <xacro:insert_block name="origin"/>
+      <xacro:insert_block name="origin" />
       <mass value="${mass}" />
       <inertia ixx="${(1/12.0) * mass * (3*radius*radius + length*length)}"
-              ixy="0.0" ixz="0.0"
-              iyy="${(1/12.0) * mass * (3*radius*radius + length*length)}"
-              iyz="0.0"
-              izz="${0.5 * mass * radius*radius}" />
+        ixy="0.0" ixz="0.0"
+        iyy="${(1/12.0) * mass * (3*radius*radius + length*length)}"
+        iyz="0.0"
+        izz="${0.5 * mass * radius*radius}" />
     </inertial>
   </xacro:macro>
@@ -30,13 +30,13 @@
     <visual>
       <geometry>
-        <box size="0.3 0.3 0.1"/>
+        <box size="0.3 0.3 0.1" />
       </geometry>
       <material>
-        <color rgba="0.8 0.8 0.8 1"/>
+        <color rgba="0.8 0.8 0.8 1" />
       </material>
     </visual>
     <collision>
       <geometry>
-        <box size="0.3 0.3 0.1"/>
+        <box size="0.3 0.3 0.1" />
       </geometry>
     </collision>
@@ -49,21 +49,21 @@
       y="0.28"
       z="0.18">
-      <origin xyz="0 0 0.09" rpy="0 0 0"/>
+      <origin xyz="0 0 0.09" rpy="0 0 0" />
     </xacro:inertial_box>
   </link>
   <!-- Odom Frame -->
-  <link name="odom"/>
+  <link name="odom" />
   <!-- Joint connecting base_link to odom -->
   <joint name="base_to_odom" type="fixed">
-    <parent link="odom"/>
-    <child link="base_link"/>
-    <origin xyz="0 0 0" rpy="0 0 0"/>
+    <parent link="odom" />
+    <child link="base_link" />
+    <origin xyz="0 0 0" rpy="0 0 0" />
   </joint>
   <link name="Body_link">
     <collision>
-        <origin xyz="0 0 0.0885" rpy="0 0 0"/>
-        <geometry>
-            <box size="0.45 0.28 0.18"/>
-        </geometry>
+      <origin xyz="0 0 0.0885" rpy="0 0 0" />
+      <geometry>
+        <box size="0.45 0.28 0.18" />
+      </geometry>
     </collision>
     <xacro:inertial_box
@@ -73,50 +73,51 @@
       z="0.18">
       <origin xyz="0 0 0.09" rpy="0 0 0" />
-  </xacro:inertial_box>
+    </xacro:inertial_box>
     <visual>
-        <origin rpy="0.0 1.42294 0.0" xyz="0.17482 -0.00088 0.15732"/>
-        <material name="Material.001"/>
-        <geometry>
-            <mesh filename="package://re4life_robot_description/meshes/Cylinder.001.dae" scale="0.00883 0.00889 0.10297"/>
-        </geometry>
+      <origin rpy="0.0 1.42294 0.0" xyz="0.17482 -0.00088 0.15732" />
+      <material name="Material.001" />
+      <geometry>
+        <mesh filename="package://re4life_robot_description/meshes/Cylinder.001.dae"
+          scale="0.00883 0.00889 0.10297" />
+      </geometry>
     </visual>
   </link>
   <joint name="base_to_body" type="fixed">
-      <parent link="base_link"/>
-      <child link="Body_link"/>
-      <origin xyz="0 0 0" rpy="0 0 0"/>
+    <parent link="base_link" />
+    <child link="Body_link" />
+    <origin xyz="0 0 0" rpy="0 0 0" />
   </joint>
   <joint name="BackWheel_link_joint" type="revolute">
-    <parent link="Body_link"/>
-    <child link="BackWheel_link"/>
-    <origin xyz="-0.45842 0.00285 0.05" rpy="${pi/2} 0 0"/>
-    <axis xyz="0 0 1"/>
-    <limit effort="5" velocity="5"/>
-    <dynamics damping="0.0" friction="0.0"/>
+    <parent link="Body_link" />
+    <child link="BackWheel_link" />
+    <origin xyz="-0.45842 0.00285 0.05" rpy="${pi/2} 0 0" />
+    <axis xyz="0 0 1" />
+    <limit effort="2000" velocity="5" />
+    <dynamics damping="0.0" friction="0.0" />
   </joint>
   <joint name="FrontWheel_link_joint" type="revolute">
-    <parent link="Body_link"/>
-    <child link="FrontWheel_link"/>
-    <origin xyz="0.17030 0.00221 0.05" rpy="${pi/2} 0 0"/>
-    <axis xyz="0 0 1"/>
-    <limit effort="5" velocity="5"/>
-    <dynamics damping="0.0" friction="0.0"/>
+    <parent link="Body_link" />
+    <child link="FrontWheel_link" />
+    <origin xyz="0.17030 0.00221 0.05" rpy="${pi/2} 0 0" />
+    <axis xyz="0 0 1" />
+    <limit effort="2000" velocity="5" />
+    <dynamics damping="0.0" friction="0.0" />
   </joint>
   <!-- Driving wheels - increased effort and adjusted dynamics -->
   <joint name="LeftWheel_link_joint" type="continuous">
-    <limit effort="250" velocity="50"/>  <!-- Increased effort from 10 to 50 -->
-    <origin rpy="${-pi/2} 0 0" xyz="-0.24508 0.28586 0.05"/>
-    <parent link="Body_link"/>
-    <child link="LeftWheel_link"/>
-    <axis xyz="0 0 1"/>
-    <dynamics damping="5.0" friction="0.1"/>
+    <limit effort="2000" velocity="10" />  <!-- Increased effort from 10 to 50 -->
+    <origin rpy="${-pi/2} 0 0" xyz="-0.24508 0.28586 0.05" />
+    <parent link="Body_link" />
+    <child link="LeftWheel_link" />
+    <axis xyz="0 0 1" />
+    <dynamics damping="0.1" friction="0.1" />
   </joint>
   <joint name="RightWheel_link_joint" type="continuous">
-    <limit effort="250" velocity="50"/>  <!-- Increased effort from 10 to 50 -->
-    <origin rpy="${pi/2} 0 0" xyz="-0.24508 -0.28586 0.05"/>
-    <parent link="Body_link"/>
-    <child link="RightWheel_link"/>
-    <axis xyz="0 0 -1"/>
-    <dynamics damping="5.0" friction="0.1"/>
+    <limit effort="2000" velocity="10" />  <!-- Increased effort from 10 to 50 -->
+    <origin rpy="${pi/2} 0 0" xyz="-0.24508 -0.28586 0.05" />
+    <parent link="Body_link" />
+    <child link="RightWheel_link" />
+    <axis xyz="0 0 -1" />
+    <dynamics damping="0.1" friction="0.1" />
   </joint>
   <!-- Wheels - increased mass from 0.5 to 3.75 kg each -->
@@ -124,20 +125,27 @@
   <link name="BackWheel_link">
     <collision>
-      <origin xyz="0 0 0" rpy="${pi/2} 0 ${pi/2}"/>
-      <geometry>
-        <cylinder radius="0.05" length="0.02"/>
-      </geometry>
-    </collision>
-    <xacro:inertial_cylinder
+      <origin xyz="0 0 0" rpy="${pi/2} 0 ${pi/2}" />
+      <geometry>
+        <cylinder radius="0.05" length="0.02" />
+      </geometry>
+    </collision>
+    <!-- <xacro:inertial_cylinder
     mass="3.75"
     length="0.02"
     radius="0.05">
     <origin xyz="-0.45842 0.00285 0.05" rpy="${pi/2} 0 0"/>
-  </xacro:inertial_cylinder>
+  </xacro:inertial_cylinder> -->
+    <xacro:inertial_cylinder
+      mass="3.75"
+      length="0.02"
+      radius="0.05">
+      <origin xyz="0 0 0" rpy="0 0 0" />
+    </xacro:inertial_cylinder>
     <visual name="BackWheel">
-      <origin xyz="0 0 0" rpy="${pi/2} 0 ${pi/2}"/>
-      <material name="Backdrop.011"/>
-      <geometry>
-        <mesh filename="package://re4life_robot_description/meshes/Front_end.012.dae" scale="0.0026 0.0026 0.0026"/>
+      <origin xyz="0 0 0" rpy="${pi/2} 0 ${pi/2}" />
+      <material name="Backdrop.011" />
+      <geometry>
+        <mesh filename="package://re4life_robot_description/meshes/Front_end.012.dae"
+          scale="0.0026 0.0026 0.0026" />
       </geometry>
     </visual>
@@ -146,20 +154,27 @@
   <link name="FrontWheel_link">
     <collision>
-      <origin xyz="0 0 0" rpy="${pi/2} 0 ${pi/2}"/>
-      <geometry>
-        <cylinder radius="0.05" length="0.02"/>
-      </geometry>
-    </collision>
-    <xacro:inertial_cylinder
+      <origin xyz="0 0 0" rpy="${pi/2} 0 ${pi/2}" />
+      <geometry>
+        <cylinder radius="0.05" length="0.02" />
+      </geometry>
+    </collision>
+    <!-- <xacro:inertial_cylinder
     mass="3.75"
     length="0.02"
     radius="0.05">
     <origin xyz="-0.45842 0.00285 0.05" rpy="${pi/2} 0 0"/>
-  </xacro:inertial_cylinder>
+  </xacro:inertial_cylinder> -->
+    <xacro:inertial_cylinder
+      mass="3.75"
+      length="0.02"
+      radius="0.05">
+      <origin xyz="0 0 0" rpy="0 0 0" />
+    </xacro:inertial_cylinder>
     <visual name="FrontWheel">
-      <origin xyz="0 0 0" rpy="${pi/2} 0 ${pi/2}"/>
-      <material name="Backdrop.010"/>
-      <geometry>
-        <mesh filename="package://re4life_robot_description/meshes/Front_end.011.dae" scale="0.0026 0.0026 0.0026"/>
+      <origin xyz="0 0 0" rpy="${pi/2} 0 ${pi/2}" />
+      <material name="Backdrop.010" />
+      <geometry>
+        <mesh filename="package://re4life_robot_description/meshes/Front_end.011.dae"
+          scale="0.0026 0.0026 0.0026" />
       </geometry>
     </visual>
@@ -168,25 +183,32 @@
   <link name="LeftWheel_link">
     <collision>
-      <origin xyz="0 0 0" rpy="${-pi/2} 0 ${pi/2}"/>
-      <geometry>
-        <cylinder radius="0.05" length="0.02"/>
+      <origin xyz="0 0 0" rpy="${-pi/2} 0 ${pi/2}" />
+      <geometry>
+        <cylinder radius="0.05" length="0.02" />
       </geometry>
     </collision>
     <visual name="LeftWheel">
-      <origin xyz="0 0 0" rpy="${-pi/2} 0 ${pi/2}"/>
-      <material name="Backdrop.013"/>
-      <geometry>
-        <mesh filename="package://re4life_robot_description/meshes/Front_end.014.dae" scale="0.0026 0.0026 0.0026"/>
-      </geometry>
-    </visual>
-    <xacro:inertial_cylinder
+      <origin xyz="0 0 0" rpy="${-pi/2} 0 ${pi/2}" />
+      <material name="Backdrop.013" />
+      <geometry>
+        <mesh filename="package://re4life_robot_description/meshes/Front_end.014.dae"
+          scale="0.0026 0.0026 0.0026" />
+      </geometry>
+    </visual>
+    <!-- <xacro:inertial_cylinder
     mass="3.75"
     length="0.02"
     radius="0.05">
     <origin xyz="-0.45842 0.00285 0.05" rpy="${pi/2} 0 0"/>
-  </xacro:inertial_cylinder>
-    <collision>
-      <geometry>
-        <cylinder radius="0.05" length="0.02"/>
+  </xacro:inertial_cylinder> -->
+    <xacro:inertial_cylinder
+      mass="3.75"
+      length="0.02"
+      radius="0.05">
+      <origin xyz="0 0 0" rpy="0 0 0" />
+    </xacro:inertial_cylinder>
+    <collision>
+      <geometry>
+        <cylinder radius="0.05" length="0.02" />
       </geometry>
       <surface>
@@ -204,25 +226,32 @@
   <link name="RightWheel_link">
     <collision>
-      <origin xyz="0 0 0" rpy="${pi/2} 0 ${pi/2}"/>
-      <geometry>
-        <cylinder radius="0.05" length="0.02"/>
+      <origin xyz="0 0 0" rpy="${pi/2} 0 ${pi/2}" />
+      <geometry>
+        <cylinder radius="0.05" length="0.02" />
       </geometry>
     </collision>
     <visual name="RightWheel">
-      <origin xyz="0 0 0" rpy="${pi/2} 0 ${pi/2}"/>
-      <material name="Backdrop.012"/>
-      <geometry>
-        <mesh filename="package://re4life_robot_description/meshes/Front_end.013.dae" scale="0.0026 0.0026 0.0026"/>
-      </geometry>
-    </visual>
-    <xacro:inertial_cylinder
+      <origin xyz="0 0 0" rpy="${pi/2} 0 ${pi/2}" />
+      <material name="Backdrop.012" />
+      <geometry>
+        <mesh filename="package://re4life_robot_description/meshes/Front_end.013.dae"
+          scale="0.0026 0.0026 0.0026" />
+      </geometry>
+    </visual>
+    <!-- <xacro:inertial_cylinder
     mass="3.75"
     length="0.02"
     radius="0.05">
     <origin xyz="-0.45842 0.00285 0.05" rpy="${pi/2} 0 0"/>
-  </xacro:inertial_cylinder>
-    <collision>
-      <geometry>
-        <cylinder radius="0.05" length="0.02"/>
+  </xacro:inertial_cylinder> -->
+    <xacro:inertial_cylinder
+      mass="3.75"
+      length="0.02"
+      radius="0.05">
+      <origin xyz="0 0 0" rpy="0 0 0" />
+    </xacro:inertial_cylinder>
+    <collision>
+      <geometry>
+        <cylinder radius="0.05" length="0.02" />
       </geometry>
       <surface>
@@ -240,51 +269,50 @@
   <link name="ultrasonic_link">
     <visual name="ultrasonic">
-      <origin rpy="0.0 0.0 0.0" xyz="0.0 0.0 0.0"/>
-      <geometry>
-        <box size="0.00334 0.00396 0.00339"/>
+      <origin rpy="0.0 0.0 0.0" xyz="0.0 0.0 0.0" />
+      <geometry>
+        <box size="0.00334 0.00396 0.00339" />
       </geometry>
     </visual>
   </link>
   <joint name="ultrasonic_link_joint" type="fixed">
-    <limit effort="30" lower="-3" upper="3" velocity="1"/>
-    <origin rpy="0 0 0" xyz="0.23943 -0.00200 0.04405"/>
-    <parent link="Body_link"/>
-    <child link="ultrasonic_link"/>
-  </joint>
-  <!-- LIDAR link - unchanged -->
+    <limit effort="30" lower="-3" upper="3" velocity="1" />
+    <origin rpy="0 0 0" xyz="0.23943 -0.00200 0.04405" />
+    <parent link="Body_link" />
+    <child link="ultrasonic_link" />
+  </joint>
   <link name="lidar_link">
     <inertial>
-      <mass value="0.5"/>  <!-- Increased from 0.05 to 0.5 kg -->
-      <origin xyz="0 0 0" rpy="0 0 0"/>
-      <inertia ixx="1e-4" ixy="0" ixz="0" iyy="1e-4" iyz="0" izz="1e-4"/>  <!-- Increased inertia -->
+      <mass value="0.5" />
+      <origin xyz="0 0 0" rpy="0 0 0" />
+      <inertia ixx="1e-4" ixy="0" ixz="0" iyy="1e-4" iyz="0" izz="1e-4" />
     </inertial>
     <visual>
-      <origin xyz="0 0 0" rpy="0 0 0"/>
-      <geometry>
-        <cylinder radius="0.03" length="0.02"/>
-      </geometry>
-    </visual>
-    <collision>
-      <origin xyz="0 0 0" rpy="0 0 0"/>
-      <geometry>
-        <cylinder radius="0.03" length="0.02"/>
+      <origin xyz="0 0 0" rpy="0 0 0" />
+      <geometry>
+        <cylinder radius="0.03" length="0.02" />
+      </geometry>
+    </visual>
+    <collision>
+      <origin xyz="0 0 0" rpy="0 0 0" />
+      <geometry>
+        <cylinder radius="0.03" length="0.02" />
       </geometry>
     </collision>
   </link>
   <joint name="lidar_joint" type="fixed">
-    <parent link="Body_link"/>
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
File: urdf/relife_ros2_control.xacro (robot description, xacro)
@@ -7,6 +7,6 @@
         <joint name="RightWheel_link_joint">
             <command_interface name="velocity">
-                <param name="min">-150.0</param>  <!-- Increased range from -1 to -2 -->
-                <param name="max">150.0</param>   <!-- Increased range from 1 to 2 -->
+                <param name="min">-150.0</param>
+                <param name="max">150.0</param>
             </command_interface>
             <state_interface name="position" />
@@ -14,9 +14,9 @@
             <parameters>
                 <pid>
-                    <p>15.0</p>    <!-- Moderately increased from 10.0 -->
-                    <i>0.2</i>     <!-- Moderately increased from 0.1 -->
-                    <d>0.02</d>    <!-- Moderately increased from 0.01 -->
-                  </pid>
-              </parameters>
+                    <p>100.0</p>
+                    <i>0.2</i>
+                    <d>0.02</d>
+                </pid>
+            </parameters>
         </joint>
         <joint name="LeftWheel_link_joint">
@@ -29,31 +29,11 @@
             <parameters>
                 <pid>
-                    <p>15.0</p>    <!-- Moderately increased from 10.0 -->
-                    <i>0.2</i>     <!-- Moderately increased from 0.1 -->
-                    <d>0.02</d>    <!-- Moderately increased from 0.01 -->
-                  </pid>
-              </parameters>
+                    <p>100.0</p>
+                    <i>0.2</i>
+                    <d>0.02</d>
+                </pid>
+            </parameters>
         </joint>
     </ros2_control>
-    <transmission name="rightwheel_transmission">
-        <type>transmission_interface/SimpleTransmission</type>
-        <actuator name="rightwheel_motor">
-            <hardwareInterface>hardware_interface/velocity</hardwareInterface>
-        </actuator>
-        <joint name="RightWheel_link_joint">
-            <hardwareInterface>hardware_interface/velocity</hardwareInterface>
-            <mechanical_reduction>2.5</mechanical_reduction>  <!-- Further reduced from 5.0 -->
-        </joint>
-    </transmission>
-    <transmission name="leftwheel_transmission">
-        <type>transmission_interface/SimpleTransmission</type>
-        <actuator name="leftwheel_motor">
-            <hardwareInterface>hardware_interface/velocity</hardwareInterface>
-        </actuator>
-        <joint name="LeftWheel_link_joint">
-            <hardwareInterface>hardware_interface/velocity</hardwareInterface>
-            <mechanical_reduction>2.5</mechanical_reduction>  <!-- Further reduced from 5.0 -->
-        </joint>
-    </transmission>
     <gazebo>
         <plugin name="gazebo_ros2_control" filename="libgazebo_ros2_control.so">
