Commit message: last changes (hopefully)

File: urdf/relife_model.urdf.xacro (robot description, xacro)
@@ -29,26 +29,22 @@
   <link name="base_link">
     <visual>
-      <geometry>
-        <box size="0.3 0.3 0.1" />
-      </geometry>
-      <material>
-        <color rgba="0.8 0.8 0.8 1" />
-      </material>
-    </visual>
-    <collision>
-      <geometry>
-        <box size="0.3 0.3 0.1" />
-      </geometry>
-    </collision>
-    <!-- <xacro:inertial_box mass="15.0" x="0.3" y="0.3" z="0.1">
-      <origin xyz="0 0 0" rpy="0 0 0"/>
-    </xacro:inertial_box> -->
+      <origin rpy="0.0 1.42294 0.0" xyz="0.17482 -0.00088 0.15732" />
+      <material name="Material.001" />
+      <geometry>
+        <mesh filename="package://re4life_robot_description/meshes/Cylinder.001.dae"
+          scale="0.00883 0.00889 0.10297" />
+      </geometry>
+    </visual>
+    <collision>
+      <origin xyz="0 0 0.15" rpy="0 0 0" /> <geometry>
+        <box size="0.45 0.28 0.18" />
+      </geometry>
+    </collision>
     <xacro:inertial_box
-      mass="85.0"
+      mass="15.0"
       x="0.45"
       y="0.28"
       z="0.18">
-      <origin xyz="0 0 0.09" rpy="0 0 0" />
-    </xacro:inertial_box>
+      <origin xyz="0 0 0.15" rpy="0 0 0" /> </xacro:inertial_box>
   </link>
   <!-- Odom Frame -->
@@ -60,7 +56,7 @@
     <origin xyz="0 0 0" rpy="0 0 0" />
   </joint>
-  <link name="Body_link">
-    <collision>
-      <origin xyz="0 0 0.0885" rpy="0 0 0" />
+  <!-- <link name="Body_link">
+    <collision>
+      <origin xyz="0 0 0.10" rpy="0 0 0" />
       <geometry>
         <box size="0.45 0.28 0.18" />
@@ -82,25 +78,25 @@
       </geometry>
     </visual>
-  </link>
-  <joint name="base_to_body" type="fixed">
+  </link> -->
+  <!-- <joint name="base_to_body" type="fixed">
     <parent link="base_link" />
     <child link="Body_link" />
     <origin xyz="0 0 0" rpy="0 0 0" />
-  </joint>
-  <joint name="BackWheel_link_joint" type="revolute">
-    <parent link="Body_link" />
+  </joint> -->
+  <joint name="BackWheel_link_joint" type="continuous">
+    <parent link="base_link" />
     <child link="BackWheel_link" />
     <origin xyz="-0.45842 0.00285 0.05" rpy="${pi/2} 0 0" />
     <axis xyz="0 0 1" />
     <limit effort="2000" velocity="5" />
-    <dynamics damping="0.0" friction="0.0" />
-  </joint>
-  <joint name="FrontWheel_link_joint" type="revolute">
-    <parent link="Body_link" />
+    <dynamics damping="0.1" friction="0.0" />
+  </joint>
+  <joint name="FrontWheel_link_joint" type="continuous">
+    <parent link="base_link" />
     <child link="FrontWheel_link" />
     <origin xyz="0.17030 0.00221 0.05" rpy="${pi/2} 0 0" />
     <axis xyz="0 0 1" />
     <limit effort="2000" velocity="5" />
-    <dynamics damping="0.0" friction="0.0" />
+    <dynamics damping="0.1" friction="0.0" />
   </joint>
   <!-- Driving wheels - increased effort and adjusted dynamics -->
@@ -108,5 +104,5 @@
     <limit effort="2000" velocity="10" />  <!-- Increased effort from 10 to 50 -->
     <origin rpy="${-pi/2} 0 0" xyz="-0.24508 0.28586 0.05" />
-    <parent link="Body_link" />
+    <parent link="base_link" />
     <child link="LeftWheel_link" />
     <axis xyz="0 0 1" />
@@ -116,5 +112,5 @@
     <limit effort="2000" velocity="10" />  <!-- Increased effort from 10 to 50 -->
     <origin rpy="${pi/2} 0 0" xyz="-0.24508 -0.28586 0.05" />
-    <parent link="Body_link" />
+    <parent link="base_link" />
     <child link="RightWheel_link" />
     <axis xyz="0 0 -1" />
@@ -125,8 +121,28 @@
   <link name="BackWheel_link">
     <collision>
-      <origin xyz="0 0 0" rpy="${pi/2} 0 ${pi/2}" />
+      <origin xyz="0 0 0" rpy="0 0 0" />
       <geometry>
         <cylinder radius="0.05" length="0.02" />
       </geometry>
+      <surface>
+        <friction>
+          <ode>
+            <mu>0.1</mu>
+            <mu2>0.1</mu2>
+            <slip1>1.0</slip1>
+            <slip2>1.0</slip2>
+          </ode>
+        </friction>
+        <contact>
+          <ode>
+            <soft_cfm>0</soft_cfm>
+            <soft_erp>0.2</soft_erp>
+            <kp>1000000.0</kp>
+            <kd>100.0</kd>
+            <max_vel>0.01</max_vel>
+            <min_depth>0.001</min_depth>
+          </ode>
+        </contact>
+      </surface>
     </collision>
     <!-- <xacro:inertial_cylinder
@@ -154,8 +170,28 @@
   <link name="FrontWheel_link">
     <collision>
-      <origin xyz="0 0 0" rpy="${pi/2} 0 ${pi/2}" />
+      <origin xyz="0 0 0" rpy="0 0 0" />
       <geometry>
         <cylinder radius="0.05" length="0.02" />
       </geometry>
+      <surface>
+        <friction>
+          <ode>
+            <mu>0.1</mu>
+            <mu2>0.1</mu2>
+            <slip1>1.0</slip1>
+            <slip2>1.0</slip2>
+          </ode>
+        </friction>
+        <contact>
+          <ode>
+            <soft_cfm>0</soft_cfm>
+            <soft_erp>0.2</soft_erp>
+            <kp>1000000.0</kp>
+            <kd>100.0</kd>
+            <max_vel>0.01</max_vel>
+            <min_depth>0.001</min_depth>
+          </ode>
+        </contact>
+      </surface>
     </collision>
     <!-- <xacro:inertial_cylinder
@@ -183,8 +219,26 @@
   <link name="LeftWheel_link">
     <collision>
-      <origin xyz="0 0 0" rpy="${-pi/2} 0 ${pi/2}" />
+      <origin xyz="0 0 0" rpy="0 0 0" />
       <geometry>
         <cylinder radius="0.05" length="0.02" />
       </geometry>
+      <surface>
+        <friction>
+          <ode>
+            <mu>0.8</mu>
+            <mu2>0.4</mu2>
+          </ode>
+        </friction>
+        <contact>
+          <ode>
+            <soft_cfm>0</soft_cfm>
+            <soft_erp>0.2</soft_erp>
+            <kp>1000000.0</kp>
+            <kd>100.0</kd>
+            <max_vel>0.01</max_vel>
+            <min_depth>0.001</min_depth>
+          </ode>
+        </contact>
+      </surface>
     </collision>
     <visual name="LeftWheel">
@@ -208,5 +262,9 @@
       <origin xyz="0 0 0" rpy="0 0 0" />
     </xacro:inertial_cylinder>
-    <collision>
+  </link>
+  <!-- Right Wheel -->
+  <link name="RightWheel_link">
+    <collision>
+      <origin xyz="0 0 0" rpy="0 0 0" />
       <geometry>
         <cylinder radius="0.05" length="0.02" />
@@ -215,19 +273,19 @@
         <friction>
           <ode>
-            <mu>0.8</mu>    <!-- sliding friction -->
-            <mu2>0.4</mu2>  <!-- rolling friction -->
+            <mu>0.8</mu>
+            <mu2>0.4</mu2>
           </ode>
         </friction>
-        <!-- optional bounce, contact parameters, etc. -->
+        <contact>
+          <ode>
+            <soft_cfm>0</soft_cfm>
+            <soft_erp>0.2</soft_erp>
+            <kp>1000000.0</kp>
+            <kd>100.0</kd>
+            <max_vel>0.01</max_vel>
+            <min_depth>0.001</min_depth>
+          </ode>
+        </contact>
       </surface>
-    </collision>
-  </link>
-  <!-- Right Wheel -->
-  <link name="RightWheel_link">
-    <collision>
-      <origin xyz="0 0 0" rpy="${pi/2} 0 ${pi/2}" />
-      <geometry>
-        <cylinder radius="0.05" length="0.02" />
-      </geometry>
     </collision>
     <visual name="RightWheel">
@@ -251,18 +309,4 @@
       <origin xyz="0 0 0" rpy="0 0 0" />
     </xacro:inertial_cylinder>
-    <collision>
-      <geometry>
-        <cylinder radius="0.05" length="0.02" />
-      </geometry>
-      <surface>
-        <friction>
-          <ode>
-            <mu>0.8</mu>    <!-- sliding friction -->
-            <mu2>0.4</mu2>  <!-- rolling friction -->
-          </ode>
-        </friction>
-        <!-- optional bounce, contact parameters, etc. -->
-      </surface>
-    </collision>
   </link>
   <!-- Ultrasonic sensor - unchanged -->
@@ -278,5 +322,5 @@
     <limit effort="30" lower="-3" upper="3" velocity="1" />
     <origin rpy="0 0 0" xyz="0.23943 -0.00200 0.04405" />
-    <parent link="Body_link" />
+    <parent link="base_link" />
     <child link="ultrasonic_link" />
   </joint>
@@ -301,5 +345,5 @@
   </link>
   <joint name="lidar_joint" type="fixed">
-    <parent link="Body_link" />
+    <parent link="base_link" />
     <child link="lidar_link" />
     <origin xyz="0 0 0.25" rpy="0 0 0" />
@@ -308,5 +352,5 @@
   <joint name="camera_joint" type="fixed">
     <origin rpy="0.0 1.5708 0.0" xyz="0.19112 0.00194 0.54940" />
-    <parent link="Body_link" />
+    <parent link="base_link" />
     <child link="camera" />
   </joint>
@@ -370,14 +414,14 @@
   </gazebo>
   <gazebo reference="FrontWheel_link">
-    <mu1>0.1</mu1>  <!-- Lowered from 0.2 for better sliding -->
-    <mu2>0.1</mu2>  <!-- Lowered from 0.2 for better sliding -->
-    <kp>10.0</kp>  <!-- Increased for better stability -->
-    <kd>10.0</kd>  <!-- Increased for better stability -->
+    <mu1>0.1</mu1>
+    <mu2>0.1</mu2>
+    <kp>1000000.0</kp>
+    <kd>100.0</kd>
   </gazebo>
   <gazebo reference="BackWheel_link">
-    <mu1>0.1</mu1>  <!-- Lowered from 0.2 for better sliding -->
-    <mu2>0.1</mu2>  <!-- Lowered from 0.2 for better sliding -->
-    <kp>10.0</kp>  <!-- Increased for better stability -->
-    <kd>10.0</kd>  <!-- Increased for better stability -->
+    <mu1>0.1</mu1>
+    <mu2>0.1</mu2>
+    <kp>1000000.0</kp>
+    <kd>100.0</kd>
   </gazebo>
   <!-- LIDAR sensor - unchanged -->
